Commit message: Add base_footprint Add dummy link for robot_state Fix rplidar frame Fix rpicam frame Fix realsense frame

File: urdf/antrobot.xacro (robot description, xacro)
@@ -4,4 +4,9 @@
 <xacro:include filename="$(find antrobot_description)/urdf/antrobot.trans" />
 <xacro:include filename="$(find antrobot_description)/urdf/antrobot.gazebo" />
+<link name="dummy"/>
+<joint name="dummy_joint" type="fixed">
+<parent link="dummy"/>
+<child link="base_link"/>
+</joint>
 <link name="base_link">
   <inertial>
@@ -24,4 +29,5 @@
   </collision>
 </link>
+<link name="base_footprint"/>
 <link name="wheel_left_link_1">
   <inertial>
@@ -71,5 +77,5 @@
   </inertial>
   <visual>
-    <origin xyz="-0.0 -0.0 -0.155" rpy="0 0 0"/>
+    <origin xyz="-0.0 -0.0 -0.186" rpy="0 0 0"/>
     <geometry>
       <mesh filename="file://$(find antrobot_description)/meshes/rplidar_link_1.stl" scale="0.001 0.001 0.001"/>
@@ -78,5 +84,5 @@
   </visual>
   <collision>
-    <origin xyz="-0.0 -0.0 -0.155" rpy="0 0 0"/>
+    <origin xyz="-0.0 -0.0 -0.186" rpy="0 0 0"/>
     <geometry>
       <mesh filename="file://$(find antrobot_description)/meshes/rplidar_link_1.stl" scale="0.001 0.001 0.001"/>
@@ -137,17 +143,22 @@
 </joint>
 <joint name="rplidar_joint" type="fixed">
-  <origin xyz="0.0 0.0 0.155" rpy="0 0 0"/>
+  <origin xyz="0.0 0.0 0.186" rpy="0 0 0"/>
   <parent link="base_link"/>
   <child link="rplidar_link_1"/>
 </joint>
 <joint name="rpicam_joint" type="fixed">
-  <origin xyz="0.126235 8.8e-05 0.031943" rpy="0 0 0"/>
+  <origin xyz="0.126235 8.8e-05 0.031943" rpy="0 0.0523599 0"/>
   <parent link="base_link"/>
   <child link="rpicam_link_1"/>
 </joint>
 <joint name="realsense_joint" type="fixed">
-  <origin xyz="0.111521 0.00012 0.132217" rpy="0 0 0"/>
+  <origin xyz="0.111521 0.00012 0.132217" rpy="0 0.0523599 0"/>
   <parent link="base_link"/>
   <child link="realsense_link_1"/>
 </joint>
+<joint name="base_footprint_joint" type="fixed">
+  <origin xyz="0 0 -0.035" rpy="0 0 0"/>
+  <parent link="base_link"/>
+  <child link="base_footprint"/>
+</joint>
 </robot>

Commit message: Add robot orgin frame for direct gazebo loading

File: urdf/antrobot.xacro (robot description, xacro)
@@ -4,9 +4,12 @@
 <xacro:include filename="$(find antrobot_description)/urdf/antrobot.trans" />
 <xacro:include filename="$(find antrobot_description)/urdf/antrobot.gazebo" />
-<link name="dummy"/>
-<joint name="dummy_joint" type="fixed">
-<parent link="dummy"/>
-<child link="base_link"/>
-</joint>
+<link name="robot_origin">
+  <visual>
+    <origin xyz="0 0 0" rpy="0 0 0"/>
+  </visual>
+  <collision>
+    <origin xyz="0 0 0" rpy="0 0 0"/>
+  </collision>
+</link>
 <link name="base_link">
   <inertial>
@@ -30,5 +33,5 @@
 </link>
 <link name="base_footprint"/>
-<link name="wheel_left_link_1">
+<link name="wheel_left_link">
   <inertial>
     <origin xyz="-1.2728583304935648e-06 -0.0023063066184155906 6.00040961839729e-08" rpy="0 0 0"/>
@@ -39,5 +42,5 @@
     <origin xyz="-0.029613 -0.1095 0.005" rpy="0 0 0"/>
     <geometry>
-      <mesh filename="file://$(find antrobot_description)/meshes/wheel_left_link_1.stl" scale="0.001 0.001 0.001"/>
+      <mesh filename="file://$(find antrobot_description)/meshes/wheel_left_link.stl" scale="0.001 0.001 0.001"/>
     </geometry>
     <material name="silver"/>
@@ -46,9 +49,9 @@
     <origin xyz="-0.029613 -0.1095 0.005" rpy="0 0 0"/>
     <geometry>
-      <mesh filename="file://$(find antrobot_description)/meshes/wheel_left_link_1.stl" scale="0.001 0.001 0.001"/>
+      <mesh filename="file://$(find antrobot_description)/meshes/wheel_left_link.stl" scale="0.001 0.001 0.001"/>
     </geometry>
   </collision>
 </link>
-<link name="wheel_right_link_1">
+<link name="wheel_right_link">
   <inertial>
     <origin xyz="1.4357516585211672e-06 0.002306307129465418 6.000408169209298e-08" rpy="0 0 0"/>
@@ -59,5 +62,5 @@
     <origin xyz="-0.029613 0.1095 0.005" rpy="0 0 0"/>
     <geometry>
-      <mesh filename="file://$(find antrobot_description)/meshes/wheel_right_link_1.stl" scale="0.001 0.001 0.001"/>
+      <mesh filename="file://$(find antrobot_description)/meshes/wheel_right_link.stl" scale="0.001 0.001 0.001"/>
     </geometry>
     <material name="silver"/>
@@ -66,9 +69,9 @@
     <origin xyz="-0.029613 0.1095 0.005" rpy="0 0 0"/>
     <geometry>
-      <mesh filename="file://$(find antrobot_description)/meshes/wheel_right_link_1.stl" scale="0.001 0.001 0.001"/>
+      <mesh filename="file://$(find antrobot_description)/meshes/wheel_right_link.stl" scale="0.001 0.001 0.001"/>
     </geometry>
   </collision>
 </link>
-<link name="rplidar_link_1">
+<link name="rplidar_link">
   <inertial>
     <origin xyz="0.0030931959904156093 -0.0003163045555262638 0.021005003394948152" rpy="0 0 0"/>
@@ -79,5 +82,5 @@
     <origin xyz="-0.0 -0.0 -0.186" rpy="0 0 0"/>
     <geometry>
-      <mesh filename="file://$(find antrobot_description)/meshes/rplidar_link_1.stl" scale="0.001 0.001 0.001"/>
+      <mesh filename="file://$(find antrobot_description)/meshes/rplidar_link.stl" scale="0.001 0.001 0.001"/>
     </geometry>
     <material name="silver"/>
@@ -86,9 +89,9 @@
     <origin xyz="-0.0 -0.0 -0.186" rpy="0 0 0"/>
     <geometry>
-      <mesh filename="file://$(find antrobot_description)/meshes/rplidar_link_1.stl" scale="0.001 0.001 0.001"/>
+      <mesh filename="file://$(find antrobot_description)/meshes/rplidar_link.stl" scale="0.001 0.001 0.001"/>
     </geometry>
   </collision>
 </link>
-<link name="rpicam_link_1">
+<link name="rpicam_link">
   <inertial>
     <origin xyz="-0.006587669853958977 5.666710231481823e-05 1.5965148283683672e-05" rpy="0 0 0"/>
@@ -99,5 +102,5 @@
     <origin xyz="-0.126235 -8.8e-05 -0.031943" rpy="0 0 0"/>
     <geometry>
-      <mesh filename="file://$(find antrobot_description)/meshes/rpicam_link_1.stl" scale="0.001 0.001 0.001"/>
+      <mesh filename="file://$(find antrobot_description)/meshes/rpicam_link.stl" scale="0.001 0.001 0.001"/>
     </geometry>
     <material name="silver"/>
@@ -106,9 +109,9 @@
     <origin xyz="-0.126235 -8.8e-05 -0.031943" rpy="0 0 0"/>
     <geometry>
-      <mesh filename="file://$(find antrobot_description)/meshes/rpicam_link_1.stl" scale="0.001 0.001 0.001"/>
+      <mesh filename="file://$(find antrobot_description)/meshes/rpicam_link.stl" scale="0.001 0.001 0.001"/>
     </geometry>
   </collision>
 </link>
-<link name="realsense_link_1">
+<link name="realsense_link">
   <inertial>
     <origin xyz="-0.012605676757880976 0.001112839462886813 0.0006324082805583275" rpy="0 0 0"/>
@@ -119,5 +122,5 @@
     <origin xyz="-0.111521 -0.00012 -0.132217" rpy="0 0 0"/>
     <geometry>
-      <mesh filename="file://$(find antrobot_description)/meshes/realsense_link_1.stl" scale="0.001 0.001 0.001"/>
+      <mesh filename="file://$(find antrobot_description)/meshes/realsense_link.stl" scale="0.001 0.001 0.001"/>
     </geometry>
     <material name="silver"/>
@@ -126,5 +129,5 @@
     <origin xyz="-0.111521 -0.00012 -0.132217" rpy="0 0 0"/>
     <geometry>
-      <mesh filename="file://$(find antrobot_description)/meshes/realsense_link_1.stl" scale="0.001 0.001 0.001"/>
+      <mesh filename="file://$(find antrobot_description)/meshes/realsense_link.stl" scale="0.001 0.001 0.001"/>
     </geometry>
   </collision>
@@ -133,5 +136,5 @@
   <origin xyz="0.029613 0.1095 -0.005" rpy="0 0 0"/>
   <parent link="base_link"/>
-  <child link="wheel_left_link_1"/>
+  <child link="wheel_left_link"/>
   <axis xyz="-0.0 1.0 -0.0"/>
 </joint>
@@ -139,5 +142,5 @@
   <origin xyz="0.029613 -0.1095 -0.005" rpy="0 0 0"/>
   <parent link="base_link"/>
-  <child link="wheel_right_link_1"/>
+  <child link="wheel_right_link"/>
   <axis xyz="0.0 -1.0 0.0"/>
 </joint>
@@ -145,15 +148,15 @@
   <origin xyz="0.0 0.0 0.186" rpy="0 0 0"/>
   <parent link="base_link"/>
-  <child link="rplidar_link_1"/>
+  <child link="rplidar_link"/>
 </joint>
 <joint name="rpicam_joint" type="fixed">
   <origin xyz="0.126235 8.8e-05 0.031943" rpy="0 0.0523599 0"/>
   <parent link="base_link"/>
-  <child link="rpicam_link_1"/>
+  <child link="rpicam_link"/>
 </joint>
 <joint name="realsense_joint" type="fixed">
   <origin xyz="0.111521 0.00012 0.132217" rpy="0 0.0523599 0"/>
   <parent link="base_link"/>
-  <child link="realsense_link_1"/>
+  <child link="realsense_link"/>
 </joint>
 <joint name="base_footprint_joint" type="fixed">
@@ -162,3 +165,8 @@
   <child link="base_footprint"/>
 </joint>
+<joint name="base_joint" type="fixed">
+<origin xyz="0 0 0.035" rpy="0 0 0"/>
+<parent link="robot_origin"/>
+<child link="base_link"/>
+</joint>
 </robot>

Commit message: Add colors to rviz and gazebo Fix robot origin visual element

File: urdf/antrobot.xacro (robot description, xacro)
@@ -7,7 +7,13 @@
   <visual>
     <origin xyz="0 0 0" rpy="0 0 0"/>
+    <geometry>
+      <box size="0.0001 0.0001 0.0001"/>
+    </geometry>
   </visual>
   <collision>
     <origin xyz="0 0 0" rpy="0 0 0"/>
+    <geometry>
+      <box size="0.0001 0.0001 0.0001"/>
+    </geometry>
   </collision>
 </link>
@@ -23,5 +29,5 @@
       <mesh filename="file://$(find antrobot_description)/meshes/base_link.stl" scale="0.001 0.001 0.001"/>
     </geometry>
-    <material name="silver"/>
+    <material name="light_grey"/>
   </visual>
   <collision>
@@ -44,5 +50,5 @@
       <mesh filename="file://$(find antrobot_description)/meshes/wheel_left_link.stl" scale="0.001 0.001 0.001"/>
     </geometry>
-    <material name="silver"/>
+    <material name="blue"/>
   </visual>
   <collision>
@@ -64,5 +70,5 @@
       <mesh filename="file://$(find antrobot_description)/meshes/wheel_right_link.stl" scale="0.001 0.001 0.001"/>
     </geometry>
-    <material name="silver"/>
+    <material name="blue"/>
   </visual>
   <collision>
@@ -84,5 +90,5 @@
       <mesh filename="file://$(find antrobot_description)/meshes/rplidar_link.stl" scale="0.001 0.001 0.001"/>
     </geometry>
-    <material name="silver"/>
+    <material name="red"/>
   </visual>
   <collision>
@@ -104,5 +110,5 @@
       <mesh filename="file://$(find antrobot_description)/meshes/rpicam_link.stl" scale="0.001 0.001 0.001"/>
     </geometry>
-    <material name="silver"/>
+    <material name="yellow"/>
   </visual>
   <collision>
@@ -124,5 +130,5 @@
       <mesh filename="file://$(find antrobot_description)/meshes/realsense_link.stl" scale="0.001 0.001 0.001"/>
     </geometry>
-    <material name="silver"/>
+    <material name="yellow"/>
   </visual>
   <collision>

File: urdf/materials.xacro (robot description, xacro)
@@ -4,3 +4,21 @@
   <color rgba="0.700 0.700 0.700 1.000"/>
 </material>
+<material name="red">
+  <color rgba="0.902 0.196 0.157 1.000"/>
+</material>
+<material name="yellow">
+  <color rgba="1 0.816 0.129 1.000"/>
+</material>
+<material name="blue">
+  <color rgba="0.251 0.424 0.969 1.000"/>
+</material>
+<material name="dark_grey">
+  <color rgba="0.341 0.361 0.431 1.000"/>
+</material>
+<material name="grey">
+  <color rgba="0.576 0.592 0.639 1.000"/>
+</material>
+<material name="light_grey">
+  <color rgba="0.788 0.812 0.878 1.000"/>
+</material>
 </robot>

Commit message: Add ign gazebo launcher Update the main xacro Update the rviz display

File: urdf/antrobot.xacro (robot description, xacro)
@@ -4,4 +4,5 @@
 <xacro:include filename="$(find antrobot_description)/urdf/antrobot.trans" />
 <xacro:include filename="$(find antrobot_description)/urdf/antrobot.gazebo" />
+<!-- This must be checked, we don't want to fix the robot to the origin -->
 <link name="robot_origin">
   <visual>
@@ -18,4 +19,14 @@
   </collision>
 </link>
+<joint name="base_joint" type="fixed">
+<origin xyz="0 0 0.035" rpy="0 0 0"/>
+<parent link="robot_origin"/>
+<child link="base_link"/>
+</joint>
+<!-- <link name="robot_origin" />
+<joint name="robot_origin" type="fixed">
+  <parent link="base_footprint" />
+  <child link="base_link" />
+</joint> -->
 <link name="base_link">
   <inertial>
@@ -171,8 +182,3 @@
   <child link="base_footprint"/>
 </joint>
-<joint name="base_joint" type="fixed">
-<origin xyz="0 0 0.035" rpy="0 0 0"/>
-<parent link="robot_origin"/>
-<child link="base_link"/>
-</joint>
 </robot>

Commit message: Add structural defitions

File: urdf/antrobot.xacro (robot description, xacro)
@@ -1,7 +1,30 @@
 <?xml version="1.0" ?>
 <robot name="antrobot" xmlns:xacro="http://www.ros.org/wiki/xacro">
+<!-- TODO: Colisions need to be updated to a simplified version -->
+<!-- TODO: Inertial can be aproximated with cilinders if the sim is slow -->
 <xacro:include filename="$(find antrobot_description)/urdf/materials.xacro" />
 <xacro:include filename="$(find antrobot_description)/urdf/antrobot.trans" />
 <xacro:include filename="$(find antrobot_description)/urdf/antrobot.gazebo" />
+<!-- the robot wheel radius in meters -->
+<xacro:property name="wheel_radius" value="0.03"/>
+<!-- the robot wheel separation (wheel base) in meters -->
+<xacro:property name="wheel_separation" value="0.219"/>
+<!-- the robot wheel x, y, z offsets  in meters from base_link-->
+<xacro:property name="wheel_x_offset" value="0.029613"/>
+<xacro:property name="wheel_y_offset" value="0.1095"/>
+<xacro:property name="wheel_z_offset" value="0.005"/>
+<!-- the robot rplidar x, y, z offsets  in meters from base_link-->
+<xacro:property name="rplidar_x_offset" value="0.0"/>
+<xacro:property name="rplidar_y_offset" value="0.0"/>
+<xacro:property name="rplidar_z_offset" value="0.186"/>
+<!-- the robot rpicam x, y, z offsets  in meters from base_link-->
+<xacro:property name="rpicam_x_offset" value="0.126235 "/>
+<xacro:property name="rpicam_y_offset" value="8.8e-05"/>
+<xacro:property name="rpicam_z_offset" value="0.031943"/>
+<!-- the robot realsense x, y, z offsets  in meters from base_link-->
+<xacro:property name="realsense_x_offset" value="0.111521"/>
+<xacro:property name="realsense_y_offset" value="0.00012"/>
+<xacro:property name="realsense_z_offset" value="0.132217"/>
+<xacro:property name="pitch_offset" value="0 0.0523599"/>
 <!-- This must be checked, we don't want to fix the robot to the origin -->
 <link name="robot_origin">
@@ -20,5 +43,5 @@
 </link>
 <joint name="base_joint" type="fixed">
-<origin xyz="0 0 0.035" rpy="0 0 0"/>
+<origin xyz="0 0 ${wheel_radius + wheel_z_offset}" rpy="0 0 0"/>
 <parent link="robot_origin"/>
 <child link="base_link"/>
@@ -57,5 +80,5 @@
   </inertial>
   <visual>
-    <origin xyz="-0.029613 -0.1095 0.005" rpy="0 0 0"/>
+    <origin xyz="-${wheel_x_offset} -${wheel_y_offset} ${wheel_z_offset}" rpy="0 0 0"/>
     <geometry>
       <mesh filename="file://$(find antrobot_description)/meshes/wheel_left_link.stl" scale="0.001 0.001 0.001"/>
@@ -64,5 +87,5 @@
   </visual>
   <collision>
-    <origin xyz="-0.029613 -0.1095 0.005" rpy="0 0 0"/>
+    <origin xyz="-${wheel_x_offset} -${wheel_y_offset} ${wheel_z_offset}" rpy="0 0 0"/>
     <geometry>
       <mesh filename="file://$(find antrobot_description)/meshes/wheel_left_link.stl" scale="0.001 0.001 0.001"/>
@@ -77,5 +100,5 @@
   </inertial>
   <visual>
-    <origin xyz="-0.029613 0.1095 0.005" rpy="0 0 0"/>
+    <origin xyz="-${wheel_x_offset} ${wheel_y_offset} ${wheel_z_offset}" rpy="0 0 0"/>
     <geometry>
       <mesh filename="file://$(find antrobot_description)/meshes/wheel_right_link.stl" scale="0.001 0.001 0.001"/>
@@ -84,5 +107,5 @@
   </visual>
   <collision>
-    <origin xyz="-0.029613 0.1095 0.005" rpy="0 0 0"/>
+    <origin xyz="-${wheel_x_offset} -${wheel_y_offset} ${wheel_z_offset}" rpy="0 0 0"/>
     <geometry>
       <mesh filename="file://$(find antrobot_description)/meshes/wheel_right_link.stl" scale="0.001 0.001 0.001"/>
@@ -97,5 +120,5 @@
   </inertial>
   <visual>
-    <origin xyz="-0.0 -0.0 -0.186" rpy="0 0 0"/>
+    <origin xyz="-${rplidar_x_offset} -${rplidar_y_offset} -${rplidar_z_offset}" rpy="0 0 0"/>
     <geometry>
       <mesh filename="file://$(find antrobot_description)/meshes/rplidar_link.stl" scale="0.001 0.001 0.001"/>
@@ -104,5 +127,5 @@
   </visual>
   <collision>
-    <origin xyz="-0.0 -0.0 -0.186" rpy="0 0 0"/>
+    <origin xyz="-${rplidar_x_offset} -${rplidar_y_offset} -${rplidar_z_offset}" rpy="0 0 0"/>
     <geometry>
       <mesh filename="file://$(find antrobot_description)/meshes/rplidar_link.stl" scale="0.001 0.001 0.001"/>
@@ -117,5 +140,5 @@
   </inertial>
   <visual>
-    <origin xyz="-0.126235 -8.8e-05 -0.031943" rpy="0 0 0"/>
+    <origin xyz="-${rpicam_x_offset} -${rpicam_y_offset} -${rpicam_z_offset}" rpy="0 0 0"/>
     <geometry>
       <mesh filename="file://$(find antrobot_description)/meshes/rpicam_link.stl" scale="0.001 0.001 0.001"/>
@@ -124,5 +147,5 @@
   </visual>
   <collision>
-    <origin xyz="-0.126235 -8.8e-05 -0.031943" rpy="0 0 0"/>
+    <origin xyz="-${rpicam_x_offset} -${rpicam_y_offset} -${rpicam_z_offset}" rpy="0 0 0"/>
     <geometry>
       <mesh filename="file://$(find antrobot_description)/meshes/rpicam_link.stl" scale="0.001 0.001 0.001"/>
@@ -137,5 +160,5 @@
   </inertial>
   <visual>
-    <origin xyz="-0.111521 -0.00012 -0.132217" rpy="0 0 0"/>
+    <origin xyz="-${realsense_x_offset} -${realsense_y_offset} -${realsense_z_offset}" rpy="0 0 0"/>
     <geometry>
       <mesh filename="file://$(find antrobot_description)/meshes/realsense_link.stl" scale="0.001 0.001 0.001"/>
@@ -144,5 +167,5 @@
   </visual>
   <collision>
-    <origin xyz="-0.111521 -0.00012 -0.132217" rpy="0 0 0"/>
+    <origin xyz="-${realsense_x_offset} -${realsense_y_offset} -${realsense_z_offset}" rpy="0 0 0"/>
     <geometry>
       <mesh filename="file://$(find antrobot_description)/meshes/realsense_link.stl" scale="0.001 0.001 0.001"/>
@@ -151,5 +174,5 @@
 </link>
 <joint name="wheel_left_joint" type="continuous">
-  <origin xyz="0.029613 0.1095 -0.005" rpy="0 0 0"/>
+  <origin xyz="${wheel_x_offset} ${wheel_y_offset} -${wheel_z_offset}" rpy="0 0 0"/>
   <parent link="base_link"/>
   <child link="wheel_left_link"/>
@@ -157,5 +180,5 @@
 </joint>
 <joint name="wheel_right_joint" type="continuous">
-  <origin xyz="0.029613 -0.1095 -0.005" rpy="0 0 0"/>
+  <origin xyz="${wheel_x_offset} -${wheel_y_offset} -${wheel_z_offset}" rpy="0 0 0"/>
   <parent link="base_link"/>
   <child link="wheel_right_link"/>
@@ -163,20 +186,20 @@
 </joint>
 <joint name="rplidar_joint" type="fixed">
-  <origin xyz="0.0 0.0 0.186" rpy="0 0 0"/>
+  <origin xyz="${rplidar_x_offset} ${rplidar_y_offset} ${rplidar_z_offset}" rpy="0 0 0"/>
   <parent link="base_link"/>
   <child link="rplidar_link"/>
 </joint>
 <joint name="rpicam_joint" type="fixed">
-  <origin xyz="0.126235 8.8e-05 0.031943" rpy="0 0.0523599 0"/>
+  <origin xyz="${rpicam_x_offset} ${rpicam_y_offset} ${rpicam_z_offset}" rpy="0 0.0523599 0"/>
   <parent link="base_link"/>
   <child link="rpicam_link"/>
 </joint>
 <joint name="realsense_joint" type="fixed">
-  <origin xyz="0.111521 0.00012 0.132217" rpy="0 0.0523599 0"/>
+  <origin xyz="${realsense_x_offset} ${realsense_y_offset} ${realsense_z_offset}" rpy="0 0.0523599 0"/>
   <parent link="base_link"/>
   <child link="realsense_link"/>
 </joint>
 <joint name="base_footprint_joint" type="fixed">
-  <origin xyz="0 0 -0.035" rpy="0 0 0"/>
+  <origin xyz="0 0 -${wheel_radius + wheel_z_offset}" rpy="0 0 0"/>
   <parent link="base_link"/>
   <child link="base_footprint"/>

Commit message: Remove unecessary link

File: urdf/antrobot.xacro (robot description, xacro)
@@ -27,29 +27,4 @@
 <xacro:property name="realsense_z_offset" value="0.132217"/>
 <xacro:property name="pitch_offset" value="0 0.0523599"/>
-<!-- This must be checked, we don't want to fix the robot to the origin -->
-<link name="robot_origin">
-  <visual>
-    <origin xyz="0 0 0" rpy="0 0 0"/>
-    <geometry>
-      <box size="0.0001 0.0001 0.0001"/>
-    </geometry>
-  </visual>
-  <collision>
-    <origin xyz="0 0 0" rpy="0 0 0"/>
-    <geometry>
-      <box size="0.0001 0.0001 0.0001"/>
-    </geometry>
-  </collision>
-</link>
-<joint name="base_joint" type="fixed">
-<origin xyz="0 0 ${wheel_radius + wheel_z_offset}" rpy="0 0 0"/>
-<parent link="robot_origin"/>
-<child link="base_link"/>
-</joint>
-<!-- <link name="robot_origin" />
-<joint name="robot_origin" type="fixed">
-  <parent link="base_footprint" />
-  <child link="base_link" />
-</joint> -->
 <link name="base_link">
   <inertial>
@@ -177,5 +152,5 @@
   <parent link="base_link"/>
   <child link="wheel_left_link"/>
-  <axis xyz="-0.0 1.0 -0.0"/>
+  <axis xyz="0.0 1.0 0.0"/>
 </joint>
 <joint name="wheel_right_joint" type="continuous">
@@ -183,5 +158,5 @@
   <parent link="base_link"/>
   <child link="wheel_right_link"/>
-  <axis xyz="0.0 -1.0 0.0"/>
+  <axis xyz="0.0 1.0 0.0"/>
 </joint>
 <joint name="rplidar_joint" type="fixed">

Commit message: Comment KDL fix, creates problem for rviz robot model

File: urdf/antrobot.xacro (robot description, xacro)
@@ -27,5 +27,11 @@
 <xacro:property name="realsense_z_offset" value="0.132217"/>
 <xacro:property name="pitch_offset" value="0 0.0523599"/>
-<link name="base_link">
+<!-- Workaround for the KDL Tree -->
+<!-- <link name="dummy"/>
+<joint name="dummy_joint" type="fixed">
+<parent link="dummy"/>
+<child link="base_link"/>
+</joint> -->
+<link name='base_link'>
   <inertial>
     <origin xyz="-0.015797588649762044 0.0004259128735104659 0.06300813597085958" rpy="0 0 0"/>
