Commit message: Update dependecies Possible fix for mesh loading

File: urdf/antrobot.xacro (robot description, xacro)
@@ -42,5 +42,5 @@
     <origin xyz="0 0 0" rpy="0 0 0"/>
     <geometry>
-      <mesh filename="file://$(find antrobot_description)/meshes/base_link.stl" scale="0.001 0.001 0.001"/>
+      <mesh filename="package://antrobot_description/meshes/base_link.stl" scale="0.001 0.001 0.001"/>
     </geometry>
     <material name="light_grey"/>
@@ -49,5 +49,5 @@
     <origin xyz="0 0 0" rpy="0 0 0"/>
     <geometry>
-      <mesh filename="file://$(find antrobot_description)/meshes/base_link.stl" scale="0.001 0.001 0.001"/>
+      <mesh filename="package://antrobot_description/meshes/base_link.stl" scale="0.001 0.001 0.001"/>
     </geometry>
   </collision>
@@ -63,5 +63,5 @@
     <origin xyz="-${wheel_x_offset} -${wheel_y_offset} ${wheel_z_offset}" rpy="0 0 0"/>
     <geometry>
-      <mesh filename="file://$(find antrobot_description)/meshes/wheel_left_link.stl" scale="0.001 0.001 0.001"/>
+      <mesh filename="package://antrobot_description/meshes/wheel_left_link.stl" scale="0.001 0.001 0.001"/>
     </geometry>
     <material name="blue"/>
@@ -70,5 +70,5 @@
     <origin xyz="-${wheel_x_offset} -${wheel_y_offset} ${wheel_z_offset}" rpy="0 0 0"/>
     <geometry>
-      <mesh filename="file://$(find antrobot_description)/meshes/wheel_left_link.stl" scale="0.001 0.001 0.001"/>
+      <mesh filename="package://antrobot_description/meshes/wheel_left_link.stl" scale="0.001 0.001 0.001"/>
     </geometry>
   </collision>
@@ -83,5 +83,5 @@
     <origin xyz="-${wheel_x_offset} ${wheel_y_offset} ${wheel_z_offset}" rpy="0 0 0"/>
     <geometry>
-      <mesh filename="file://$(find antrobot_description)/meshes/wheel_right_link.stl" scale="0.001 0.001 0.001"/>
+      <mesh filename="package://antrobot_description/meshes/wheel_right_link.stl" scale="0.001 0.001 0.001"/>
     </geometry>
     <material name="blue"/>
@@ -90,5 +90,5 @@
     <origin xyz="-${wheel_x_offset} -${wheel_y_offset} ${wheel_z_offset}" rpy="0 0 0"/>
     <geometry>
-      <mesh filename="file://$(find antrobot_description)/meshes/wheel_right_link.stl" scale="0.001 0.001 0.001"/>
+      <mesh filename="package://antrobot_description/meshes/wheel_right_link.stl" scale="0.001 0.001 0.001"/>
     </geometry>
   </collision>
@@ -103,5 +103,5 @@
     <origin xyz="-${rplidar_x_offset} -${rplidar_y_offset} -${rplidar_z_offset}" rpy="0 0 0"/>
     <geometry>
-      <mesh filename="file://$(find antrobot_description)/meshes/rplidar_link.stl" scale="0.001 0.001 0.001"/>
+      <mesh filename="package://antrobot_description/meshes/rplidar_link.stl" scale="0.001 0.001 0.001"/>
     </geometry>
     <material name="red"/>
@@ -110,5 +110,5 @@
     <origin xyz="-${rplidar_x_offset} -${rplidar_y_offset} -${rplidar_z_offset}" rpy="0 0 0"/>
     <geometry>
-      <mesh filename="file://$(find antrobot_description)/meshes/rplidar_link.stl" scale="0.001 0.001 0.001"/>
+      <mesh filename="package://antrobot_description/meshes/rplidar_link.stl" scale="0.001 0.001 0.001"/>
     </geometry>
   </collision>
@@ -123,5 +123,5 @@
     <origin xyz="-${rpicam_x_offset} -${rpicam_y_offset} -${rpicam_z_offset}" rpy="0 0 0"/>
     <geometry>
-      <mesh filename="file://$(find antrobot_description)/meshes/rpicam_link.stl" scale="0.001 0.001 0.001"/>
+      <mesh filename="package://antrobot_description/meshes/rpicam_link.stl" scale="0.001 0.001 0.001"/>
     </geometry>
     <material name="yellow"/>
@@ -130,5 +130,5 @@
     <origin xyz="-${rpicam_x_offset} -${rpicam_y_offset} -${rpicam_z_offset}" rpy="0 0 0"/>
     <geometry>
-      <mesh filename="file://$(find antrobot_description)/meshes/rpicam_link.stl" scale="0.001 0.001 0.001"/>
+      <mesh filename="package://antrobot_description/meshes/rpicam_link.stl" scale="0.001 0.001 0.001"/>
     </geometry>
   </collision>
@@ -143,5 +143,5 @@
     <origin xyz="-${realsense_x_offset} -${realsense_y_offset} -${realsense_z_offset}" rpy="0 0 0"/>
     <geometry>
-      <mesh filename="file://$(find antrobot_description)/meshes/realsense_link.stl" scale="0.001 0.001 0.001"/>
+      <mesh filename="package://antrobot_description/meshes/realsense_link.stl" scale="0.001 0.001 0.001"/>
     </geometry>
     <material name="yellow"/>
@@ -150,5 +150,5 @@
     <origin xyz="-${realsense_x_offset} -${realsense_y_offset} -${realsense_z_offset}" rpy="0 0 0"/>
     <geometry>
-      <mesh filename="file://$(find antrobot_description)/meshes/realsense_link.stl" scale="0.001 0.001 0.001"/>
+      <mesh filename="package://antrobot_description/meshes/realsense_link.stl" scale="0.001 0.001 0.001"/>
     </geometry>
   </collision>
@@ -172,5 +172,5 @@
 </joint>
 <joint name="rpicam_joint" type="fixed">
-  <origin xyz="${rpicam_x_offset} ${rpicam_y_offset} ${rpicam_z_offset}" rpy="0 0.0523599 0"/>
+  <origin xyz="${rpicam_x_offset} ${rpicam_y_offset} ${rpicam_z_offset}" rpy="0 0 0.0523599 0"/>
   <parent link="base_link"/>
   <child link="rpicam_link"/>

Commit message: Fix rpicam joint

File: urdf/antrobot.xacro (robot description, xacro)
@@ -26,5 +26,5 @@
 <xacro:property name="realsense_y_offset" value="0.00012"/>
 <xacro:property name="realsense_z_offset" value="0.132217"/>
-<xacro:property name="pitch_offset" value="0 0.0523599"/>
+<!-- <xacro:property name="pitch_offset" value="0 0.0523599"/> -->
 <!-- Workaround for the KDL Tree -->
 <!-- <link name="dummy"/>
@@ -172,5 +172,5 @@
 </joint>
 <joint name="rpicam_joint" type="fixed">
-  <origin xyz="${rpicam_x_offset} ${rpicam_y_offset} ${rpicam_z_offset}" rpy="0 0 0.0523599 0"/>
+  <origin xyz="${rpicam_x_offset} ${rpicam_y_offset} ${rpicam_z_offset}" rpy="0 0.0523599 0"/>
   <parent link="base_link"/>
   <child link="rpicam_link"/>

Commit message: Remove transmission from old gazebo

File: urdf/antrobot.xacro (robot description, xacro)
@@ -4,5 +4,6 @@
 <!-- TODO: Inertial can be aproximated with cilinders if the sim is slow -->
 <xacro:include filename="$(find antrobot_description)/urdf/materials.xacro" />
-<xacro:include filename="$(find antrobot_description)/urdf/antrobot.trans" />
+<!-- This left over from gazebo classic not needed in gazbo ignition -->
+<!-- <xacro:include filename="$(find antrobot_description)/urdf/antrobot.trans" /> -->
 <xacro:include filename="$(find antrobot_description)/urdf/antrobot.gazebo" />
 <!-- the robot wheel radius in meters -->
@@ -88,5 +89,5 @@
   </visual>
   <collision>
-    <origin xyz="-${wheel_x_offset} -${wheel_y_offset} ${wheel_z_offset}" rpy="0 0 0"/>
+    <origin xyz="-${wheel_x_offset} ${wheel_y_offset} ${wheel_z_offset}" rpy="0 0 0"/>
     <geometry>
       <mesh filename="package://antrobot_description/meshes/wheel_right_link.stl" scale="0.001 0.001 0.001"/>
